File: Thor.kicad_pcb (KiCad board)
At the start: 2 copper layers, 39 parts, among them J1 Conn_02x32_Counter_Clockwise, J2 Conn_02x32_Counter_Clockwise, J3 Conn_01x01, J4 Conn_01x01, Q1 PHP79NQ08LT, Q2 PHP79NQ08LT, Q3 PHP79NQ08LT, Q4 PHP79NQ08LT, Q5 PHP79NQ08LT, Q6 PHP79NQ08LT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

Commit message: PCB Control Traces and Better Layout
Parts:
- added C17: 22pF, Capacitor_SMD:C_0201_0603Metric, F.Cu at (139.7, 174.0)
- J2: footprint Connector_PinHeader_2.54mm:PinHeader_2x32_P2.54mm_Horizontal -> Connector_PinSocket_2.54mm:PinSocket_2x32_P2.54mm_Horizontal
- moved J2 83.0 mm to (19.1, 111.8), turned to 0 degrees
- moved C3 81.8 mm to (174.0, 160.0)
- moved C15 74.1 mm to (36.8, 106.0), turned to 270 degrees
- moved C9 73.2 mm to (140.3, 106.0), turned to 270 degrees
- moved R3 72.6 mm to (160.0, 138.4)
- moved R4 72.6 mm to (167.6, 138.4)
- moved C4 68.9 mm to (180.3, 160.0), turned to 270 degrees
- moved C5 67.9 mm to (174.0, 154.9), turned to 270 degrees
- moved D1 64.8 mm to (180.3, 153.7)
- moved R2 61.9 mm to (149.9, 147.3)
- moved U1 61.5 mm to (163.8, 153.7)
- moved C7 57.1 mm to (48.9, 106.0), turned to 270 degrees
- moved R1 56.0 mm to (149.9, 168.9), turned to 90 degrees
- moved C16 52.7 mm to (125.7, 106.0), turned to 270 degrees
- moved RV1 51.7 mm to (139.7, 157.5), turned to 180 degrees
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Connections:
- net Net-(C10-Pad1) renamed /MainPowerBus24V
- net Net-(C12-Pad1) renamed /OutPutPowerBus
- net Net-(C5-Pad1) renamed /SwitchingBus24V
Routing:
- net Net-(C4-Pad1): track 0.00 -> 152.8 mm
- net /OutPutPowerBus: track 0.00 -> 112.3 mm, vias 0 -> 2
- net Net-(R2-Pad1): track 0.00 -> 106.8 mm
- net Net-(Q1-Pad1): track 0.00 -> 67.3 mm, vias 0 -> 1
- net Net-(RV1-Pad2): track 0.00 -> 64.8 mm
- net Net-(Q2-Pad1): track 0.00 -> 64.0 mm, vias 0 -> 1
- net Net-(C17-Pad1): track 0.00 -> 37.5 mm
- net GND: track 0.00 -> 33.4 mm, vias 0 -> 3
- net Net-(C3-Pad2): track 0.00 -> 24.0 mm
- net Net-(D1-Pad1): track 0.00 -> 15.8 mm
- net Net-(R3-Pad2): track 0.00 -> 13.8 mm
- net /MainPowerBus24V: track 0.00 -> 8.67 mm
- net Net-(C1-Pad1): track 0.00 -> 8.65 mm
- net /SwitchingBus24V: track 0.00 -> 7.90 mm
- added copper zone on B.Cu, net GND
Other:
- board outline added: 316.2 x 227.3 mm
- copper layers 2 -> 4
- net class HIGHPOWER added: clearance 0.2, trace_width 31, via_dia 0.8, via_drill 0.4

Commit message: Fixed connectors in PCB
Parts:
- J1: footprint Connector_PinHeader_2.54mm:PinHeader_2x32_P2.54mm_Horizontal -> ThorPSU:HP DPS connector
- J2: footprint Connector_PinSocket_2.54mm:PinSocket_2x32_P2.54mm_Horizontal -> ThorPSU:HP DPS connector
- moved J1 50.5 mm to (22.5, 55.0)
- moved J2 30.3 mm to (23.4, 141.7)
Connections:
- net /MainPowerBus24V renamed Net-(C10-Pad1)
- net /OutPutPowerBus renamed Net-(C12-Pad1)
- net /SwitchingBus24V renamed Net-(C5-Pad1)
Routing:
- net Net-(C12-Pad1): vias 2 -> 1
- net /OutPutPowerBus: vias 0 -> 1

Commit message: Card Connector Change and Locations Changed
Parts:
- moved R5 17.0 mm to (40.0, 175.3), turned to 90 degrees
- moved R7 16.5 mm to (33.0, 175.3), turned to 90 degrees
- moved J1 14.9 mm to (24.1, 69.8)
- moved J2 10.7 mm to (24.1, 152.4)
Routing:
- net Net-(C5-Pad1): track 7.90 -> 110.4 mm, vias 0 -> 1
- net Net-(C10-Pad1): track 8.67 -> 49.8 mm
- net Net-(J2-Pad32): track 0.00 -> 6.98 mm
- net Net-(J1-Pad32): track 0.00 -> 6.35 mm
- net Net-(J1-Pad13): track 0.00 -> 6.35 mm
Other:
- board size 316.2 x 227.3 mm -> 300 x 200 mm
Changed lines of the file:
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@@
     (thickness 1.6)
     (drawings 4)
-    (tracks 136)
+    (tracks 157)
     (zones 0)
     (modules 40)
@@
   )
   (module Resistor_THT:R_Box_L8.4mm_W2.5mm_P5.08mm (layer F.Cu)
-    (at 32.385 160.02 270)
+    (at 40.005 175.26 90)
     (descr "Resistor, Box series, Radial, pin pitch=5.08mm, 0.5W = 1/2W, length*width=8.38*2.54mm^2, http://www.vishay.com/docs/60051/cns020.pdf")
     (tags "Resistor Box series Radial pin pitch 5.08mm 0.5W = 1/2W length 8.38mm width 2.54mm")
@@
     (fp_line (start -1.65 1.27) (end 6.73 1.27) (layer F.Fab) (width 0.1))
     (fp_line (start -1.65 -1.27) (end -1.65 1.27) (layer F.Fab) (width 0.1))
-    (pad 2 thru_hole circle (at 5.08 0 270) (size 1.6 1.6) (drill 0.8) (layers *.Cu *.Mask)
+    (pad 2 thru_hole circle (at 5.08 0 90) (size 1.6 1.6) (drill 0.8) (layers *.Cu *.Mask)
       (net 2 GND))
-    (pad 1 thru_hole circle (at 0 0 270) (size 1.6 1.6) (drill 0.8) (layers *.Cu *.Mask)
+    (pad 1 thru_hole circle (at 0 0 90) (size 1.6 1.6) (drill 0.8) (layers *.Cu *.Mask)
       (net 31 "Net-(J2-Pad32)"))
     (model ${KISYS3DMOD}/Resistor_THT.3dshapes/R_Box_L8.4mm_W2.5mm_P5.08mm.wrl
@@
   )
   (module Resistor_THT:R_Box_L8.4mm_W2.5mm_P5.08mm (layer F.Cu)
-    (at 39.37 160.02 270)
+    (at 33.02 175.26 90)
     (descr "Resistor, Box series, Radial, pin pitch=5.08mm, 0.5W = 1/2W, length*width=8.38*2.54mm^2, http://www.vishay.com/docs/60051/cns020.pdf")
     (tags "Resistor Box series Radial pin pitch 5.08mm 0.5W = 1/2W length 8.38mm width 2.54mm")
@@
       (effects (font (size 1 1) (thickness 0.15)))
     )
-    (pad 1 thru_hole circle (at 0 0 270) (size 1.6 1.6) (drill 0.8) (layers *.Cu *.Mask)
+    (pad 1 thru_hole circle (at 0 0 90) (size 1.6 1.6) (drill 0.8) (layers *.Cu *.Mask)
       (net 31 "Net-(J2-Pad32)"))
-    (pad 2 thru_hole circle (at 5.08 0 270) (size 1.6 1.6) (drill 0.8) (layers *.Cu *.Mask)
+    (pad 2 thru_hole circle (at 5.08 0 90) (size 1.6 1.6) (drill 0.8) (layers *.Cu *.Mask)
       (net 2 GND))
     (model ${KISYS3DMOD}/Resistor_THT.3dshapes/R_Box_L8.4mm_W2.5mm_P5.08mm.wrl
@@
   )
   (module "ThorPSU:HP DPS connector" (layer F.Cu)
-    (at 22.5 55 180)
+    (at 24.13 69.85 180)
     (fp_text reference J1 (at 0 48.26) (layer F.SilkS)
       (effects (font (size 1 1) (thickness 0.15)))
@@
   )
   (module "ThorPSU:HP DPS connector" (layer F.Cu)
-    (at 23.4 141.7)
+    (at 24.13 152.4)
     (fp_text reference J2 (at 0 48.26) (layer F.SilkS)
       (effects (font (size 1 1) (thickness 0.15)))
@@
       (net 32 "Net-(J2-Pad33)"))
   )
-  (gr_line (start -3.81 227.33) (end -12.7 0) (layer Edge.Cuts) (width 0.05))
-  (gr_line (start 303.53 227.33) (end -3.81 227.33) (layer Edge.Cuts) (width 0.05))
-  (gr_line (start 303.53 1.27) (end 303.53 227.33) (layer Edge.Cuts) (width 0.05))
-  (gr_line (start -12.7 0) (end 303.53 1.27) (layer Edge.Cuts) (width 0.05))
+  (gr_line (start 10 205) (end 10 5) (layer Edge.Cuts) (width 0.05))
+  (gr_line (start 310 205) (end 10 205) (layer Edge.Cuts) (width 0.05))
+  (gr_line (start 310 5) (end 310 205) (layer Edge.Cuts) (width 0.05))
+  (gr_line (start 10 5) (end 310 5) (layer Edge.Cuts) (width 0.05))
   (segment (start 141.21 163.83) (end 149.86 163.83) (width 0.25) (layer F.Cu) (net 1))
   (segment (start 139.22 168.7325) (end 139.3975 168.91) (width 0.25) (layer F.Cu) (net 2))
@@
   (segment (start 180.34 152.62) (end 177.58 149.86) (width 0.25) (layer F.Cu) (net 6))
   (segment (start 180.34 152.67) (end 180.34 152.62) (width 0.25) (layer F.Cu) (net 6))
+  (segment (start 37.465 67.945) (end 31.115 67.945) (width 0.25) (layer In2.Cu) (net 16))
+  (segment (start 37.465 73.025) (end 31.115 73.025) (width 0.25) (layer In2.Cu) (net 23))
+  (segment (start 33.02 175.26) (end 40.005 175.26) (width 0.25) (layer In2.Cu) (net 31))
   (segment (start 158.75 97.79) (end 158.75 109.22) (width 0.25) (layer In1.Cu) (net 39))
   (segment (start 158.75 109.22) (end 158.75 120.65) (width 0.25) (layer In1.Cu) (net 39))
@@
   (segment (start 159.0675 155.8925) (end 161.23 155.8925) (width 0.25) (layer F.Cu) (net 43))
   (segment (start 156.21 158.75) (end 159.0675 155.8925) (width 0.25) (layer F.Cu) (net 43))
+  (segment (start 242.57 99.06) (end 242.57 99.06) (width 0.25) (layer In2.Cu) (net 46))
+  (via (at 242.57 99.06) (size 0.8) (drill 0.4) (layers F.Cu B.Cu) (net 46))
   (segment (start 173.1675 152.7175) (end 173.99 153.54) (width 0.25) (layer F.Cu) (net 47))
   (segment (start 166.43 152.7175) (end 173.1675 152.7175) (width 0.25) (layer F.Cu) (net 47))
+  (segment (start 173.99 153.54) (end 176.4 151.13) (width 0.25) (layer F.Cu) (net 47))
+  (segment (start 176.4 151.13) (end 176.4 151.13) (width 0.25) (layer F.Cu) (net 47))
+  (via (at 176.4 151.13) (size 0.8) (drill 0.4) (layers F.Cu B.Cu) (net 47))
+  (segment (start 182.88 144.65) (end 182.88 120.65) (width 0.25) (layer In1.Cu) (net 47))
+  (segment (start 176.4 151.13) (end 182.88 144.65) (width 0.25) (layer In1.Cu) (net 47))
+  (segment (start 182.88 120.65) (end 182.88 107.95) (width 0.25) (layer In1.Cu) (net 47))
+  (segment (start 182.88 107.95) (end 182.88 97.79) (width 0.25) (layer In1.Cu) (net 47))
+  (segment (start 181.602499 96.464999) (end 165.155001 96.464999) (width 0.25) (layer In1.Cu) (net 47))
+  (segment (start 182.88 97.79) (end 182.88 97.7425) (width 0.25) (layer In1.Cu) (net 47))
+  (segment (start 182.88 97.7425) (end 181.602499 96.464999) (width 0.25) (layer In1.Cu) (net 47))
+  (segment (start 165.155001 96.464999) (end 163.83 97.79) (width 0.25) (layer In1.Cu) (net 47))
+  (segment (start 163.83 97.79) (end 163.83 109.22) (width 0.25) (layer In1.Cu) (net 47))
+  (segment (start 163.83 109.22) (end 163.83 120.65) (width 0.25) (layer In1.Cu) (net 47))
   (segment (start 36.83 106.045) (end 37.88 106.045) (width 0.25) (layer F.Cu) (net 48))
   (segment (start 160.02 138.43) (end 167.64 138.43) (width 0.25) (layer F.Cu) (net 48))
+  (segment (start 160.02 138.43) (end 160.02 128.27) (width 0.25) (layer In2.Cu) (net 48))
+  (segment (start 161.29 127) (end 161.29 120.65) (width 0.25) (layer In2.Cu) (net 48))
+  (segment (start 160.02 128.27) (end 161.29 127) (width 0.25) (layer In2.Cu) (net 48))
+  (segment (start 161.29 97.79) (end 161.29 109.22) (width 0.25) (layer In2.Cu) (net 48))
+  (segment (start 161.29 109.22) (end 161.29 120.65) (width 0.25) (layer In2.Cu) (net 48))
   (segment (start 149.715001 142.384999) (end 189.085001 142.384999) (width 0.25) (layer In2.Cu) (net 49))
   (segment (start 139.7 152.4) (end 149.715001 142.384999) (width 0.25) (layer In2.Cu) (net 49))
-  (segment (start 242.57 99.06) (end 242.57 99.06) (width 0.25) (layer In2.Cu) (net 46))
-  (via (at 242.57 99.06) (size 0.8) (drill 0.4) (layers F.Cu B.Cu) (net 46))
   (segment (start 189.085001 142.384999) (end 229.725001 142.384999) (width 0.25) (layer In2.Cu) (net 49))
   (segment (start 229.725001 142.384999) (end 242.57 129.54) (width 0.25) (layer In2.Cu) (net 49))
@@
     (polygon
       (pts
-        (xy -24.13 241.3) (xy -26.67 -7.62) (xy 320.04 -6.35) (xy 312.42 237.49)
+        (xy 392.43 267.97) (xy 394.97 -31.75) (xy -92.71 -41.91) (xy -78.74 254)
       )
     )

Commit message: first complete layout with BIG Polygons
Parts:
- added C18: 0.1uF, Capacitor_SMD:C_0805_2012Metric, F.Cu at (155.6, 88.4)
- moved C17 82.4 mm to (154.1, 92.8), turned to 270 degrees
- moved C2 77.6 mm to (155.6, 92.8), turned to 270 degrees
- moved R1 75.3 mm to (150.4, 93.6), turned to 270 degrees
- moved C1 66.7 mm to (154.2, 98.7), turned to 0 degrees
- moved C3 66.3 mm to (165.8, 94.2)
- moved RV1 62.8 mm to (159.7, 97.9), turned to 90 degrees
- moved C4 62.6 mm to (177.6, 97.5)
- moved L2 62.6 mm to (220.1, 60.1)
- moved Q1 62.6 mm to (156.0, 58.1)
- moved Q2 62.6 mm to (177.6, 35.3)
- moved Q3 62.6 mm to (156.0, 35.3)
- moved Q4 62.6 mm to (177.6, 58.1)
- moved C12 62.6 mm to (279.2, 44.8)
- moved C14 62.6 mm to (255.1, 44.8)
- moved C5 62.6 mm to (171.2, 92.4)
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Connections:
- net Net-(C10-Pad1) renamed /MainPowerBus24V
- net Net-(C17-Pad1) renamed /Ith
- net Net-(C3-Pad2) renamed /Vin
- net Net-(C4-Pad1) renamed /FCB
- net Net-(C5-Pad1) renamed /SW
- net Net-(D1-Pad1) renamed /BOOST
- net Net-(J1-Pad31) renamed /PSU1_act
- net Net-(J1-Pad32) renamed /PSU_V_adjust
- net Net-(J2-Pad31) renamed /PSU2_act
- net Net-(J2-Pad32) renamed /PSU2_adj
- net Net-(Q1-Pad1) renamed /TG
- net Net-(Q2-Pad1) renamed /BG
- net Net-(R3-Pad2) renamed /Ion
- net Net-(RV1-Pad2) renamed /Vfb
- C12 pad 1: Net-(C12-Pad1) -> /OutPutPowerBus
- C14 pad 1: Net-(C12-Pad1) -> /OutPutPowerBus
- J1 pad 13: Net-(J1-Pad13) -> /12V_IN
- J1 pad 14: Net-(J1-Pad13) -> /12V_IN
- J1 pad 15: Net-(J1-Pad13) -> /12V_IN
- J1 pad 16: Net-(J1-Pad13) -> /12V_IN
- J1 pad 17: Net-(J1-Pad13) -> /12V_IN
- J1 pad 18: Net-(J1-Pad13) -> /12V_IN
- J1 pad 19: Net-(J1-Pad13) -> /12V_IN
- J1 pad 20: Net-(J1-Pad13) -> /12V_IN
- J1 pad 21: Net-(J1-Pad13) -> /12V_IN
- J1 pad 22: Net-(J1-Pad13) -> /12V_IN
- J1 pad 23: Net-(J1-Pad13) -> /12V_IN
- J1 pad 24: Net-(J1-Pad13) -> /12V_IN
- J1 pad 41: Net-(J1-Pad41) -> /12V_IN
- J1 pad 42: Net-(J1-Pad41) -> /12V_IN
- J1 pad 43: Net-(J1-Pad41) -> /12V_IN
- J1 pad 44: Net-(J1-Pad41) -> /12V_IN
- J1 pad 45: Net-(J1-Pad41) -> /12V_IN
- J1 pad 46: Net-(J1-Pad41) -> /12V_IN
- J1 pad 47: Net-(J1-Pad41) -> /12V_IN
- J1 pad 48: Net-(J1-Pad41) -> /12V_IN
- J1 pad 49: Net-(J1-Pad41) -> /12V_IN
- J1 pad 50: Net-(J1-Pad41) -> /12V_IN
- J1 pad 51: Net-(J1-Pad41) -> /12V_IN
- J1 pad 52: Net-(J1-Pad41) -> /12V_IN
- J2 pad 1: Net-(J1-Pad13) -> /12V_IN
- J2 pad 10: Net-(J1-Pad13) -> /12V_IN
- J2 pad 11: Net-(J1-Pad13) -> /12V_IN
- J2 pad 12: Net-(J1-Pad13) -> /12V_IN
- J2 pad 2: Net-(J1-Pad13) -> /12V_IN
- J2 pad 3: Net-(J1-Pad13) -> /12V_IN
- J2 pad 4: Net-(J1-Pad13) -> /12V_IN
- J2 pad 5: Net-(J1-Pad13) -> /12V_IN
- J2 pad 53: Net-(J1-Pad41) -> /12V_IN
- J2 pad 54: Net-(J1-Pad41) -> /12V_IN
- J2 pad 55: Net-(J1-Pad41) -> /12V_IN
- J2 pad 56: Net-(J1-Pad41) -> /12V_IN
- J2 pad 57: Net-(J1-Pad41) -> /12V_IN
- J2 pad 58: Net-(J1-Pad41) -> /12V_IN
- J2 pad 59: Net-(J1-Pad41) -> /12V_IN
- J2 pad 6: Net-(J1-Pad13) -> /12V_IN
- J2 pad 60: Net-(J1-Pad41) -> /12V_IN
- J2 pad 61: Net-(J1-Pad41) -> /12V_IN
- J2 pad 62: Net-(J1-Pad41) -> /12V_IN
- J2 pad 63: Net-(J1-Pad41) -> /12V_IN
- J2 pad 64: Net-(J1-Pad41) -> /12V_IN
- J2 pad 7: Net-(J1-Pad13) -> /12V_IN
- J2 pad 8: Net-(J1-Pad13) -> /12V_IN
- J2 pad 9: Net-(J1-Pad13) -> /12V_IN
- J3 pad 1: Net-(C12-Pad1) -> /OutPutPowerBus
- L1 pad 2: Net-(C12-Pad1) -> /OutPutPowerBus
- L2 pad 1: Net-(C12-Pad1) -> /OutPutPowerBus
- R2 pad 1: Net-(R2-Pad1) -> /Pgood
- R6 pad 2: Net-(J1-Pad13) -> /12V_IN
- R8 pad 2: Net-(J1-Pad13) -> /12V_IN
- RV1 pad 3: Net-(C12-Pad1) -> /OutPutPowerBus
- U1 pad 1: Net-(U1-Pad1) -> /RUNSS
- U1 pad 2: Net-(R2-Pad1) -> /Pgood
- U1 pad 3: Net-(U1-Pad3) -> GND
- U1 pad 9: Net-(R2-Pad1) -> Net-(U1-Pad9)
Routing:
- net /OutPutPowerBus: track 0.00 -> 149.9 mm, vias 1 -> 2
- net /FCB: track 152.8 -> 36.2 mm
- net Net-(C12-Pad1): track 112.3 -> 0.00 mm, vias 1 -> 0
- net Net-(R2-Pad1): track 106.8 -> 0.00 mm
- net /Vfb: track 64.8 -> 6.04 mm
- net /Ith: track 37.5 -> 8.91 mm
- net GND: track 33.4 -> 5.24 mm, vias 3 -> 90
- net /Pgood: track 0.00 -> 13.2 mm
- net /Vin: track 24.0 -> 11.8 mm, vias 0 -> 1
- net Net-(J1-Pad13): track 6.35 -> 0.00 mm
- net /PSU_V_adjust: track 6.35 -> 0.00 mm
- net Net-(C1-Pad1): track 8.65 -> 2.93 mm
- net /Ion: track 13.8 -> 9.39 mm, vias 0 -> 1
- net /RUNSS: track 0.00 -> 2.22 mm
- net /MainPowerBus24V: track 49.8 -> 51.1 mm
- added copper zone on F.Cu, net /MainPowerBus24V
- added copper zone on F.Cu, net /OutPutPowerBus
- added copper zone on F.Cu, net /SW
- added copper zone on F.Cu, net GND
- removed copper zone on B.Cu, net GND

Commit message: Form factor change
Parts:
- moved J3 242.5 mm to (57.1, 92.3), turned to 180 degrees
- moved J4 237.3 mm to (57.1, 74.9), turned to 0 degrees
- moved C15 207.0 mm to (228.1, 146.1), turned to 0 degrees
- moved C12 205.8 mm to (77.7, 86.6), turned to 90 degrees
- moved C7 191.4 mm to (228.1, 134.0), turned to 0 degrees
- moved C13 175.2 mm to (228.1, 121.3), turned to 0 degrees
- moved J1 168.1 mm to (189.4, 33.2), turned to 270 degrees
- moved C8 159.4 mm to (228.1, 108.6), turned to 0 degrees
- moved C14 158.9 mm to (101.8, 86.6), turned to 90 degrees
- moved R8 151.1 mm to (167.8, 53.9), turned to 90 degrees
- moved R6 145.9 mm to (162.8, 53.9)
- moved C11 142.6 mm to (228.1, 94.6), turned to 0 degrees
- moved J2 137.5 mm to (99.2, 32.9), turned to 270 degrees
- moved C10 128.7 mm to (228.1, 82.5), turned to 0 degrees
- moved R7 127.4 mm to (74.6, 54.9)
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Routing:
- net /SW: track 110.4 -> 56.3 mm
- net GND: track 5.24 -> 50.1 mm, vias 90 -> 91
- net /PSU_V_adjust: track 0.00 -> 34.3 mm
- net /PSU2_adj: track 6.98 -> 36.1 mm
- net /MainPowerBus24V: track 51.1 -> 24.2 mm
- net /OutPutPowerBus: track 149.9 -> 124.5 mm
- net /TG: track 67.3 -> 79.1 mm
- net /PSU1_act: track 0.00 -> 2.54 mm
- net /PSU2_act: track 0.00 -> 2.54 mm
- net /BG: track 64.0 -> 66.5 mm
- added copper zone on F.Cu, net /12V_IN
- added copper zone on B.Cu, net GND
Other:
- board size 300 x 200 mm -> 185 x 130 mm
